File: K_PSU_filter.kicad_pcb (KiCad board)
At the start: 2 copper layers, 100 x 50 mm, 32 parts, among them J1 Conn_01x02_Socket, J2 Conn_01x02_Socket

Commit message: gerber added, small silkmask mods
Parts:
- added G***: LOGO, boutfiltre:boutfiltre, B.Cu at (145.4, 56.3)

Commit message: small routing mods, new gerber, inductors are in the same direct.
Parts:
- moved L1 17.5 mm to (109.8, 66.2), turned to 45 degrees
- moved L2 15.0 mm to (126.0, 50.0), turned to -135 degrees
Routing:
- net Net-(J1-Pin_1): track 40.2 -> 23.9 mm
- net Net-(C10-Pad2): track 131.1 -> 147.2 mm
- net Net-(J1-Pin_2): track 19.2 -> 34.0 mm
- net Net-(C1-Pad1): track 127.5 -> 113.3 mm
